File: IR_AC.kicad_pcb (KiCad board)
At the start: 2 copper layers, 20 x 15 mm, 1 part

Commit message: late night work on led current
Parts:
- added C1: 1u, Capacitor_SMD:C_0603_1608Metric, F.Cu at (163.0, 63.2)
- added C2: 1u, Capacitor_SMD:C_0603_1608Metric, F.Cu at (163.0, 65.8)
- added CLDO1: 1u, Capacitor_SMD:C_0805_2012Metric, F.Cu at (127.1, 105.7)
- added CLDO2: 1u, Capacitor_SMD:C_0805_2012Metric, F.Cu at (127.1, 108.8)
- added D1: 1N5819HW, LC_libz_foot:1N5819HW, F.Cu at (131.9, 105.7)
- added D2: RED_GREEN, LED_SMD:LED_0805_2012Metric, F.Cu at (122.6, 105.8)
- added D3: RED_GREEN, LED_SMD:LED_0805_2012Metric, F.Cu at (122.6, 108.8)
- added D4: LED, LC_libz_foot:IR_LED_TH_5MM, F.Cu at (116.9, 107.8)
- added H1: MountingHole, MountingHole:MountingHole_3.2mm_M3, F.Cu at (157.0, 66.0)
- added H2: MountingHole, MountingHole:MountingHole_3.2mm_M3, F.Cu at (157.0, 73.9)
- added H3: MountingHole, MountingHole:MountingHole_3.2mm_M3, F.Cu at (157.0, 81.9)
- added H4: MountingHole, MountingHole:MountingHole_3.2mm_M3, F.Cu at (157.0, 89.8)
- added J1: TYPE-C 16PIN 2MD(073), LC_libz_foot:USB-C-SMD_TYPE-C-6PIN-2MD-073, F.Cu at (158.5, 108.7)
- added Q1: NPN, Package_TO_SOT_SMD:SOT-23, F.Cu at (131.7, 109.7)
- added R2: 10k, Resistor_SMD:R_0603_1608Metric, F.Cu at (163.0, 70.8)
- added RCC1: 5.1k, Resistor_SMD:R_0603_1608Metric, F.Cu at (163.0, 73.3)
- added RCC2: 5.1k, Resistor_SMD:R_0603_1608Metric, F.Cu at (163.0, 75.8)
- added RLED1: 220R, Resistor_SMD:R_0603_1608Metric, F.Cu at (163.0, 78.3)
- added RLED2: 820R, Resistor_SMD:R_0603_1608Metric, F.Cu at (163.0, 80.8)
- added RLED3: 330R, Resistor_SMD:R_0603_1608Metric, F.Cu at (163.0, 83.3)
- added SW1: SW_Push, LC_libz_foot:BTN_L45_W45, F.Cu at (157.7, 96.7)
- added SW2: SW_Push, LC_libz_foot:BTN_L45_W45, F.Cu at (157.7, 102.4)
- added TP1: TestPoint, TestPoint:TestPoint_THTPad_D1.5mm_Drill0.7mm, F.Cu at (105.8, 106.0)
- added TP2: TestPoint, TestPoint:TestPoint_THTPad_D1.5mm_Drill0.7mm, F.Cu at (105.8, 109.6)
- added TP3: TestPoint, TestPoint:TestPoint_THTPad_D1.5mm_Drill0.7mm, F.Cu at (105.8, 113.1)
- added U1: AP2112K-3.3TRG1, LC_libz_foot:AP2112K-3.3, F.Cu at (137.0, 106.6)
- added U2: LED-SMD_4P-L5.0-W5.0-BL_XL-5050RGBC, LC_libz_foot:WS2812B_5050, F.Cu at (110.7, 109.3)
- added U3: ESP32-S3-WROOM-1, RF_Module:ESP32-S3-WROOM-1, F.Cu at (128.5, 90.3)
- moved R1 38.2 mm to (163.0, 68.3)
Connections:
- R1 pad 1: +5V -> EN
- R1 pad 2: GND -> +3V3
Routing:
- removed copper zone on F.Cu, net +5V
- removed copper zone on F.Cu, net GND
Other:
- board outline removed
- board text removed: "AI Fusion Tensor Processor Edge Device for IoT"

Commit message: Finished schematic
Parts:
- added D4: PRTR5V0U2X, libs:SOT-666-6_L1.6-W1.2-P0.50-LS1.6-BR, F.Cu at (191.0, 73.5)
- added D6: RED, LED_SMD:LED_0805_2012Metric, F.Cu at (187.2, 73.5)
- added J2: Conn_01x04_Pin, libs:HDR-TH_4P-P2.54-V-M, F.Cu at (186.6, 65.5)
- added Q1: NMOS, Package_TO_SOT_SMD:SOT-23, F.Cu at (187.4, 69.8)
- added R4: 330R, Resistor_SMD:R_0603_1608Metric, F.Cu at (182.9, 68.7)
- added R7: 100R, Resistor_SMD:R_0603_1608Metric, F.Cu at (182.9, 71.2)
- added R8: 100k, Resistor_SMD:R_0603_1608Metric, F.Cu at (182.9, 73.7)
- added U4: USBLC6-4, libs:SOT-23-6_L2.9-W1.6-P0.95-LS2.8-BL, F.Cu at (187.1, 109.3)
- D2, D3: value RED_GREEN -> GREEN
- R1: renamed from RLED1; value 220R -> 680R
- R2: renamed from RLED2; value 820R -> 2k2
- R3: renamed from RLED3; value 330R -> 30R; footprint Resistor_SMD:R_0603_1608Metric -> Resistor_SMD:R_1206_3216Metric
- U2: value LED-SMD_4P-L5.0-W5.0-BL_XL-5050RGBC -> WS2812B_5050
- renumbered D4 to D5, R1 to R5, R2 to R6
Connections:
- net Net-(J1-CC1) renamed /CC1
- net Net-(J1-CC2) renamed /CC2
- CLDO1 pad 1: +5V -> VDC
- D1 pad 1: +5V -> VDC
- D1 pad 2: VDC -> /V_BUS
- D5 pad 1: Net-(D4-K) -> Net-(D5-K)
- J1 pad 11: VDC -> /V_BUS
- J1 pad 13: unconnected-(J1-SHELL-Pad13) -> GND
- J1 pad 14: unconnected-(J1-SHELL-Pad14) -> GND
- J1 pad 2: VDC -> /V_BUS
- J1 pad 5: D- -> Net-(J1-DN1)
- J1 pad 6: D+ -> Net-(J1-DP1)
- J1 pad 7: D- -> Net-(J1-DN1)
- J1 pad 8: D+ -> Net-(J1-DP1)
- R2 pad 2: +5V -> VDC
- R3 pad 2: +5V -> VDC
- TP1 pad 1: Net-(D2-A) -> +3V3
- TP2 pad 1: Net-(D3-A) -> VDC
- U1 pad 1: +5V -> VDC
- U1 pad 3: +5V -> VDC
- U2 pad 1: LED_STATUS -> VDC
- U2 pad 4: unconnected-(U2-DIN-Pad4) -> LED_STATUS
- U3 pad 20: unconnected-(U3-IO12-Pad20) -> LED_STATUS
- U3 pad 21: unconnected-(U3-IO13-Pad21) -> IR_LED_DRIVE
- U3 pad 36: unconnected-(U3-RXD0-Pad36) -> RX
- U3 pad 37: unconnected-(U3-TXD0-Pad37) -> TX
